Commit message: modified myrobot blabal

File: Virtual_Field_Robot_Event/my_robot/my_robot_description_fre/urdf/jackal.urdf.xacro (robot description, xacro)
@@ -1,4 +1,4 @@
 <?xml version="1.0"?>
-<robot name="jackal" xmlns:xacro="http://www.ros.org/wiki/xacro">
+<robot name="my_robot" xmlns:xacro="http://www.ros.org/wiki/xacro">
   <xacro:property name="PI" value="3.1415926535897931" />
   <xacro:property name="wheelbase" value="0.262" />
@@ -22,5 +22,5 @@
         <origin xyz="0 0 0" rpy="${PI/2} 0 0"/>
         <geometry>
-          <mesh filename="package://jackal_description_fre/meshes/jackal-wheel.stl"/>
+          <mesh filename="package://my_robot_description_fre/meshes/jackal-wheel.stl"/>
         </geometry>
         <material name="black" />
@@ -90,5 +90,5 @@
       <origin xyz="0 0 ${footprint_vertical_offset}" rpy="${PI/2} 0 ${PI/2}"/>
       <geometry>
-        <mesh filename="package://jackal_description_fre/meshes/jackal-base.stl"/>
+        <mesh filename="package://my_robot_description_fre/meshes/jackal-base.stl"/>
       </geometry>
       <material name="dark_grey" />
@@ -115,5 +115,5 @@
       <visual>
         <geometry>
-          <mesh filename="package://jackal_description_fre/meshes/jackal-fender.stl"/>
+          <mesh filename="package://my_robot_description_fre/meshes/jackal-fender.stl"/>
         </geometry>
         <material name="yellow" />
@@ -125,5 +125,5 @@
       <visual>
         <geometry>
-          <mesh filename="package://jackal_description_fre/meshes/accessory_fender.stl"/>
+          <mesh filename="package://my_robot_description_fre/meshes/accessory_fender.stl"/>
         </geometry>
         <material name="yellow" />
@@ -146,5 +146,5 @@
       <visual>
         <geometry>
-          <mesh filename="package://jackal_description_fre/meshes/jackal-fender.stl"/>
+          <mesh filename="package://my_robot_description_fre/meshes/jackal-fender.stl"/>
         </geometry>
         <material name="yellow" />
@@ -156,5 +156,5 @@
       <visual>
         <geometry>
-          <mesh filename="package://jackal_description_fre/meshes/accessory_fender.stl"/>
+          <mesh filename="package://my_robot_description_fre/meshes/accessory_fender.stl"/>
         </geometry>
         <material name="yellow" />
@@ -222,11 +222,11 @@
   </joint>
   <!-- Bring in simulation data for Gazebo. -->
-  <xacro:include filename="$(find jackal_description_fre)/urdf/jackal.gazebo" />
+  <xacro:include filename="$(find my_robot_description_fre)/urdf/jackal.gazebo" />
   <!-- Optional standard accessories, including their simulation data. The rendering
        of these into the final description is controlled by optenv variables, which
        default each one to off.-->
-  <xacro:include filename="$(find jackal_description_fre)/urdf/accessories.urdf.xacro" />
+  <xacro:include filename="$(find my_robot_description_fre)/urdf/accessories.urdf.xacro" />
   <!-- Optional custom includes. -->
-  <!--xacro:include filename="$(optenv JACKAL_URDF_EXTRAS /home/user/catkin_ws/src/FieldRobotEvent/Virtual_Field_Robot_Event/jackal_fre/jackal_description_fre/urdf/realsense.urdf.xacro)" /-->
-  <!--xacro:include filename="$(optenv JACKAL_URDF_EXTRAS /home/user/catkin_ws/src/FieldRobotEvent/Virtual_Field_Robot_Event/jackal_fre/jackal_description_fre/urdf/realsense2.urdf.xacro)" /-->
+  <!--xacro:include filename="$(optenv JACKAL_URDF_EXTRAS /home/user/catkin_ws/src/FieldRobotEvent/Virtual_Field_Robot_Event/my_robot_fre/my_robot_description_fre/urdf/realsense.urdf.xacro)" /-->
+  <!--xacro:include filename="$(optenv JACKAL_URDF_EXTRAS /home/user/catkin_ws/src/FieldRobotEvent/Virtual_Field_Robot_Event/my_robot_fre/my_robot_description_fre/urdf/realsense2.urdf.xacro)" /-->
 </robot>
